Commit message: fixed stuff

File: urdf/advanced_quadrotor.urdf (robot description, URDF)
Before this commit: robot advanced_quadrotor, 29 links, 28 joints
Links:
- link base_link: geometry collision box size=0.3 0.3 0.03; visual box size=0.3 0.3 0.03
- link guard1: geometry collision cylinder length=0.001 radius=0.18; visual cylinder length=0.001 radius=0.18
- link guard2: geometry collision cylinder length=0.001 radius=0.18; visual cylinder length=0.001 radius=0.18
- link guard3: geometry collision cylinder length=0.001 radius=0.18; visual cylinder length=0.001 radius=0.18
- link guard4: geometry collision cylinder length=0.001 radius=0.18; visual cylinder length=0.001 radius=0.18
- link motor1: geometry collision cylinder length=0.02 radius=0.01; visual cylinder length=0.02 radius=0.01
- link motor2: geometry collision cylinder length=0.02 radius=0.01; visual cylinder length=0.02 radius=0.01
- link motor3: geometry collision cylinder length=0.02 radius=0.01; visual cylinder length=0.02 radius=0.01
- link motor4: geometry collision cylinder length=0.02 radius=0.01; visual cylinder length=0.02 radius=0.01
- link propeller1: geometry collision cylinder length=0.001 radius=0.06; visual cylinder length=0.001 radius=0.06
- link propeller2: geometry collision cylinder length=0.001 radius=0.06; visual cylinder length=0.001 radius=0.06
- link propeller3: geometry collision cylinder length=0.001 radius=0.06; visual cylinder length=0.001 radius=0.06
- link propeller4: geometry collision cylinder length=0.001 radius=0.06; visual cylinder length=0.001 radius=0.06
